File: PCB/robotArm.sch (KiCad schematic (older format))
At the start: 80 parts, among them J1 Motor_eje_X, J10 Gripper, J11 Conector Auxiliar 2, J12 5v, J13 End-Stop-X, J14 End-Stop-Y, J15 End-Stop-Z, J16 jumperLed5v, J17 Conector Auxiliar 1, J18 Pulsador Externo, J2 3.3v, J20 jumperLedVcc, J21 Vcc, J3 Motor_eje_Y, J4 Motor_eje_Z, J5 micro pasos X, J6 micro pasos Y, J7 micro pasos Z, J8 Conector I2C, J9 jumperLed3.3v, Q1 BC558, Q2 BC558, Q3 BC558, SW1 RESET, SW2 STOP_EM, U1 YAAJ_BluePill, U2 LM7805_TO220, U3 LM317_TO-220

Commit message: Se actualizaron los cambios
Connections:
- net +3V3: no longer J17.1 (Pin_1), J8.1 (Pin_1)
- net +5V: now also J17.1 (Pin_1), J8.1 (Pin_1)
Changed lines of the file:
@@
 Connection ~ 6500 4550
 Wire Wire Line
-	6350 4750 6350 4950
+	6350 4750 6350 4800
 Wire Wire Line
 	6500 4600 6350 4750
@@
 L power:GNDREF #PWR013
 U 1 1 646CE458
-P 6350 4950
-F 0 "#PWR013" H 6350 4700 50  0001 C CNN
-F 1 "GNDREF" H 6355 4777 50  0000 C CNN
-F 2 "" H 6350 4950 50  0001 C CNN
-F 3 "" H 6350 4950 50  0001 C CNN
-	1    6350 4950
+P 6250 4950
+F 0 "#PWR013" H 6250 4700 50  0001 C CNN
+F 1 "GNDREF" H 6255 4777 50  0000 C CNN
+F 2 "" H 6250 4950 50  0001 C CNN
+F 3 "" H 6250 4950 50  0001 C CNN
+	1    6250 4950
 	1    0    0    -1
 $EndComp
@@
 	0    1    -1   0
 $EndComp
-Wire Wire Line
-	7100 2800 7100 2700
-Wire Wire Line
-	7150 2850 7100 2800
 $Comp
 L power:+3.3V #PWR0119
 U 1 1 66580344
-P 7100 2700
-F 0 "#PWR0119" H 7100 2550 50  0001 C CNN
-F 1 "+3.3V" H 7115 2873 50  0000 C CNN
-F 2 "" H 7100 2700 50  0001 C CNN
-F 3 "" H 7100 2700 50  0001 C CNN
-	1    7100 2700
+P 7300 3150
+F 0 "#PWR0119" H 7300 3000 50  0001 C CNN
+F 1 "+3.3V" H 7315 3323 50  0000 C CNN
+F 2 "" H 7300 3150 50  0001 C CNN
+F 3 "" H 7300 3150 50  0001 C CNN
+	1    7300 3150
 	-1   0    0    -1
 $EndComp
@@
 	8000 1150 8250 1150
 Wire Wire Line
-	7350 2850 7400 2800
-Wire Wire Line
-	7400 2800 7400 2750
-Wire Wire Line
-	7150 2850 7300 2850
-Wire Wire Line
-	7300 2750 7300 2850
-Connection ~ 7300 2850
-Wire Wire Line
-	7300 2850 7350 2850
-Wire Wire Line
 	2300 6350 2400 6350
 Wire Wire Line
@@
 	6750 2750 6750 2850
 Wire Wire Line
-	7050 2850 7100 2800
-Wire Wire Line
-	6900 2850 7050 2850
-Connection ~ 7100 2800
+	6900 2850 6950 2850
 Wire Wire Line
 	6850 2950 7050 2950
@@
 Text GLabel 6800 3400 0    50   Input ~ 0
 wait
-Text GLabel 6800 3550 0    50   Input ~ 0
-finish
 Text GLabel 6800 3700 0    50   Input ~ 0
 home
@@
 	7450 3700 7500 3750
 Wire Wire Line
-	6800 3550 7350 3550
-Wire Wire Line
 	7350 3550 7400 3600
 Wire Wire Line
@@
 Wire Wire Line
 	3050 2000 3050 2050
+$Comp
+L power:+5V #PWR?
+U 1 1 652A63E1
+P 7000 2700
+F 0 "#PWR?" H 7000 2550 50  0001 C CNN
+F 1 "+5V" H 7015 2873 50  0000 C CNN
+F 2 "" H 7000 2700 50  0001 C CNN
+F 3 "" H 7000 2700 50  0001 C CNN
+	1    7000 2700
+	1    0    0    -1
+$EndComp
+Wire Wire Line
+	6950 2850 7000 2800
+Wire Wire Line
+	7000 2800 7000 2700
+Wire Wire Line
+	7000 2800 7250 2800
+Wire Wire Line
+	7250 2800 7300 2750
+Connection ~ 7000 2800
+Wire Wire Line
+	7300 3150 7350 3150
+Wire Wire Line
+	7350 3150 7400 3100
+Wire Wire Line
+	7400 2750 7400 3100
+Wire Wire Line
+	6800 3550 7350 3550
+Text GLabel 6800 3550 0    50   Input ~ 0
+finish
+Wire Wire Line
+	6250 4950 6250 4900
+Wire Wire Line
+	6250 4900 6350 4800
 $EndSCHEMATC
