File: PCB/robotArm.kicad_pcb (KiCad board)
At the start: 2 copper layers, 85 parts, among them J1 Motor_eje_X, J10 Gripper, J11 Conector Auxiliar 2, J12 5v, J13 End-Stop-X, J14 End-Stop-Y, J15 End-Stop-Z, J16 jumperLed5v, J17 Conector Auxiliar 1, J18 jumperLedVbat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

Commit message: update interface
Parts:
- removed C1: 103, Capacitor_THT:C_Disc_D8.0mm_W2.5mm_P5.00mm
- removed C6: 470uF, Capacitor_THT:CP_Radial_D8.0mm_P3.80mm
- removed D12: LED_Vbat, LED_THT:LED_D5.0mm
- removed D13, D4, D5, D6, D7, D8, D9: 1N4007, Diode_THT:D_DO-41_SOD81_P10.16mm_Horizontal
- removed J19: Vbat, TerminalBlock:TerminalBlock_bornier-2_P5.08mm
- removed R10: 220, Resistor_THT:R_Axial_DIN0207_L6.3mm_D2.5mm_P10.16mm_Horizontal
- added C19: 103, Capacitor_THT:C_Disc_D8.0mm_W2.5mm_P5.00mm, F.Cu at (170.7, 86.8)
- added C20: 103, Capacitor_THT:C_Disc_D8.0mm_W2.5mm_P5.00mm, F.Cu at (168.8, 73.0)
- added R16: 1k, Resistor_THT:R_Axial_DIN0207_L6.3mm_D2.5mm_P10.16mm_Horizontal, F.Cu at (239.3, 101.8)
- added R17: 1k, Resistor_THT:R_Axial_DIN0207_L6.3mm_D2.5mm_P10.16mm_Horizontal, F.Cu at (235.7, 101.7)
- added R18: 1k, Resistor_THT:R_Axial_DIN0207_L6.3mm_D2.5mm_P10.16mm_Horizontal, F.Cu at (232.1, 101.7)
- added R19: 10k, Resistor_THT:R_Axial_DIN0207_L6.3mm_D2.5mm_P10.16mm_Horizontal, F.Cu at (173.1, 93.0)
- added SW2: STOP_EM, Button_Switch_THT:SW_PUSH_6mm_H5mm, F.Cu at (166.6, 106.2)
- C11, C8: value 470uF -> 10uF
- C5: value 47uF -> 10uF
- D1: value 1N4007 -> LED_Home; footprint Diode_THT:D_DO-41_SOD81_P10.16mm_Horizontal -> LED_THT:LED_D5.0mm
- D2: value 1N4007 -> LED_Wait; footprint Diode_THT:D_DO-41_SOD81_P10.16mm_Horizontal -> LED_THT:LED_D5.0mm
- D3: value 1N4007 -> LED_Finish; footprint Diode_THT:D_DO-41_SOD81_P10.16mm_Horizontal -> LED_THT:LED_D5.0mm
- J18: value jumperLedVbat -> Pulsador Externo; footprint Connector_PinHeader_2.54mm:PinHeader_2x01_P2.54mm_Vertical -> Connector_PinHeader_2.54mm:PinHeader_1x02_P2.54mm_Vertical
- J5, J6, J7: footprint Connector_PinSocket_2.54mm:PinSocket_2x03_P2.54mm_Vertical -> Connector_PinHeader_2.54mm:PinHeader_2x03_P2.54mm_Vertical
- R12, R13, R7: value 10k -> 47k
- R2, R3, R4: value 10k -> 4.7k
- SW1: value SW_Push -> RESET
- moved D1 174.9 mm to (229.9, 132.3), turned to 0 degrees
- moved D2 148.2 mm to (230.0, 118.1), turned to 0 degrees
- moved J9 128.1 mm to (256.1, 119.8), turned to 180 degrees
- moved R5 127.0 mm to (182.0, 69.7), turned to 270 degrees
- moved D3 124.6 mm to (229.9, 125.4), turned to 0 degrees
- moved R7 122.0 mm to (206.4, 128.3)
- moved D10 121.8 mm to (250.5, 120.5), turned to 270 degrees
- moved R1 121.0 mm to (252.7, 116.8)
- moved C5 120.4 mm to (244.5, 123.1)
- moved C7 114.9 mm to (249.9, 127.2), turned to 270 degrees
- moved J2 113.8 mm to (245.3, 132.2)
- moved C9 110.8 mm to (223.6, 133.7)
- moved J16 109.1 mm to (214.3, 126.7)
- moved R2 108.2 mm to (192.0, 59.8)
- moved J12 107.6 mm to (218.6, 132.4)
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Connections:
- A1 pad 14: Net-(A1-Pad14) -> Net-(A1-Pad13)
- A1 pad 9: Net-(A1-Pad9) -> EnableMotor
- A2 pad 14: Net-(A2-Pad14) -> Net-(A2-Pad13)
- A2 pad 9: Net-(A2-Pad9) -> EnableMotor
- A3 pad 14: Net-(A3-Pad14) -> Net-(A3-Pad13)
- A3 pad 9: Net-(A3-Pad9) -> EnableMotor
- D1 pad 1: Net-(A1-Pad9) -> GNDREF
- D1 pad 2: EnableMotor -> Net-(D1-Pad2)
- D2 pad 1: Net-(A2-Pad9) -> GNDREF
- D2 pad 2: EnableMotor -> Net-(D2-Pad2)
- D3 pad 1: Net-(A3-Pad9) -> GNDREF
- D3 pad 2: EnableMotor -> Net-(D3-Pad2)
- J17 pad 2: Net-(J17-Pad2) -> +3V3
- J17 pad 9: Net-(J17-Pad9) -> GNDREF
- J18 pad 1: Net-(D12-Pad2) -> GNDREF
- J18 pad 2: +BATT -> STOP
- J5 pad 1: Net-(A1-Pad12) -> Net-(A1-Pad10)
- J5 pad 2: GNDREF -> +3V3
- J5 pad 4: GNDREF -> +3V3
- J5 pad 5: Net-(A1-Pad10) -> Net-(A1-Pad12)
- J5 pad 6: GNDREF -> +3V3
- J6 pad 1: Net-(A2-Pad12) -> Net-(A2-Pad10)
- J6 pad 2: GNDREF -> +3V3
- J6 pad 4: GNDREF -> +3V3
- J6 pad 5: Net-(A2-Pad10) -> Net-(A2-Pad12)
- J6 pad 6: GNDREF -> +3V3
- J7 pad 1: Net-(A3-Pad12) -> Net-(A3-Pad10)
- J7 pad 2: GNDREF -> +3V3
- J7 pad 4: GNDREF -> +3V3
- J7 pad 5: Net-(A3-Pad10) -> Net-(A3-Pad12)
- J7 pad 6: GNDREF -> +3V3
- R12 pad 1: StopX -> StopY
- R12 pad 2: GNDREF -> +3V3
- R13 pad 2: GNDREF -> +3V3
- R7 pad 1: StopY -> StopX
- R7 pad 2: GNDREF -> +3V3
- U1 pad 10: Net-(J17-Pad4) -> Net-(J17-Pad3)
- U1 pad 11: Net-(J17-Pad3) -> home
- U1 pad 12: Net-(J17-Pad2) -> finish
- U1 pad 13: SleepMotor -> wait
- U1 pad 21: +BATT -> Net-(U1-Pad21)
- U1 pad 4: ResetMotor -> STOP
- U1 pad 5: Net-(J17-Pad9) -> Net-(J17-Pad8)
- U1 pad 6: Net-(J17-Pad8) -> Net-(J17-Pad7)
- U1 pad 7: Net-(J17-Pad7) -> Net-(J17-Pad6)
- U1 pad 8: Net-(J17-Pad6) -> Net-(J17-Pad5)
- U1 pad 9: Net-(J17-Pad5) -> Net-(J17-Pad4)
Routing:
- net SleepMotor: track 126.1 -> 0.00 mm
- net ResetMotor: track 91.6 -> 0.00 mm
- net +BATT: track 57.5 -> 0.00 mm, vias 2 -> 0
- net STOP: track 0.00 -> 51.1 mm
- net home: track 0.00 -> 46.4 mm
- net finish: track 0.00 -> 37.4 mm
- net Net-(A2-Pad13): track 35.7 -> 7.55 mm
- net wait: track 0.00 -> 28.0 mm
- net Net-(C20-Pad1): track 27.5 -> 51.6 mm
- net Net-(D1-Pad2): track 0.00 -> 23.2 mm
- net DirZ: track 80.8 -> 58.0 mm
- net Net-(A3-Pad13): track 28.2 -> 7.24 mm
- net Net-(D3-Pad2): track 0.00 -> 14.8 mm
- net +5V: track 130.7 -> 118.7 mm
- net +3V3: track 411.1 -> 420.8 mm, vias 6 -> 4
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Other:
- board text added: "V:1.5 F:11/9/2023"
- board text removed: "V:1.0 F:22/6/2023"

Commit message: Se actualizaron los cambios
Connections:
- J17 pad 1: +3V3 -> +5V
- J8 pad 1: +3V3 -> +5V
Routing:
- net +5V: track 118.7 -> 136.3 mm, vias 2 -> 4
- net Net-(J8-Pad3): track 8.18 -> 10.2 mm
- net Net-(J8-Pad2): track 8.18 -> 9.88 mm
- net +3V3: track 420.8 -> 420.2 mm
Other:
- board text added: "V:1.6 F:12/10/2023"
- board text removed: "V:1.5 F:11/9/2023"

Commit message: return 2025
Parts:
- added H1: MountingHole, MountingHole:MountingHole_3.2mm_M3_DIN965, F.Cu at (258.5, 42.5)
- added H2: MountingHole, MountingHole:MountingHole_3.2mm_M3_DIN965, F.Cu at (165.0, 40.5)
- added H3: MountingHole, MountingHole:MountingHole_3.2mm_M3_DIN965, F.Cu at (258.5, 134.0)
- added H4: MountingHole, MountingHole:MountingHole_3.2mm_M3_DIN965, F.Cu at (166.0, 135.0)
- J12, J2: footprint TerminalBlock:TerminalBlock_bornier-2_P5.08mm -> TerminalBlock_Phoenix:TerminalBlock_Phoenix_PT-1,5-2-5.0-H_1x02_P5.00mm_Horizontal
- J21: footprint TerminalBlock:TerminalBlock_bornier-2_P5.08mm -> TerminalBlock_Phoenix:TerminalBlock_Phoenix_MKDS-1,5-2_1x02_P5.00mm_Horizontal
- moved C20 27.0 mm to (179.0, 98.0), turned to 90 degrees
- moved C19 13.8 mm to (166.5, 100.0)
- moved J21 5.15 mm to (259.0, 54.0), turned to 90 degrees
- moved J2 5.01 mm to (240.3, 132.0), turned to 0 degrees
- moved J12 4.62 mm to (214.0, 133.0), turned to 0 degrees
- moved A3 0.07 mm to (242.5, 52.5)
- moved A1 0.05 mm to (185.9, 52.0)
Connections:
- D18 pad 2: Net-(D18-Pad2) -> Net-(D18-A)
- J12 pad 1: +5V -> GNDREF
- J12 pad 2: GNDREF -> +5V
- J2 pad 1: +3V3 -> GNDREF
- J2 pad 2: GNDREF -> +3V3
- J21 pad 1: GNDREF -> Net-(D18-A)
- J21 pad 2: Net-(D18-Pad2) -> GNDREF
- U1 pad 21: Net-(U1-Pad21) -> unconnected-(U1-VBat-Pad21)
- U1 pad 22: Net-(U1-Pad22) -> unconnected-(U1-PC13-Pad22)
- U1 pad 23: Net-(U1-Pad23) -> unconnected-(U1-PC14-Pad23)
- U1 pad 24: Net-(U1-Pad24) -> unconnected-(U1-PC15-Pad24)
Routing:
- net Net-(U1-RST): track 51.6 -> 57.6 mm
- net Net-(D18-Pad2): track 5.06 -> 0.00 mm
- net Net-(D18-A): track 0.00 -> 5.06 mm
- net VCC: track 185.4 -> 182.5 mm
- net STOP: track 51.1 -> 49.5 mm
Other:
- board outline added: 100 x 100 mm
- net class Default removed
